File: pcb/thesensor.kicad_pcb (KiCad board)
At the start: 2 copper layers, 56.1 x 66.3 mm, 16 parts, among them J1 BME680, J3 ST7789, J5 Battery, J6 UPS, SW1 SW_SPDT, U1 XIAO-ESP32-C6-DIP

Commit message: overhaul the schematic and change pcb a bit
Parts:
- added D1: 1N4004, Diode_THT:D_DO-41_SOD81_P10.16mm_Horizontal, F.Cu at (104.0, 45.9)
- moved R1 25.3 mm to (103.8, 62.2)
- moved J3 8.86 mm to (86.4, 30.0)
- moved R2 1.08 mm to (103.8, 49.2)
- moved G*** 0.76 mm to (84.2, 54.5)
- moved NEXT1 0.76 mm to (93.3, 74.5)
- moved SELECT1 0.76 mm to (72.6, 74.5)
- moved SW1 0.51 mm to (85.0, 23.4)
- moved J6 0.37 mm to (116.3, 55.9)
Connections:
- net Net-(J1-SCL) renamed D5
- net Net-(J1-SDA) renamed D4
- net Net-(J3-BLK) renamed D2
- net Net-(J3-CS) renamed D7
- net Net-(J3-DC) renamed D9
- net Net-(J3-RES) renamed D1
- net Net-(J3-SCL) renamed D8
- net Net-(J3-SDA) renamed D10
- net Net-(J5-B+) renamed B+
- net Net-(U1-PA02_A0_D0) renamed D0
- net Net-(U1-PA11_A3_D3) renamed D3
- net Net-(U1-PB08_A6_D6_TX) renamed D6
- J1 pad 1: Net-(J1-VCC) -> 3V3
- J3 pad 2: Net-(J1-VCC) -> 3V3
- SW1 pad 2: Net-(J1-VCC) -> Net-(D1-A)
- U1 pad 12: Net-(J1-VCC) -> 3V3
- U1 pad 14: unconnected-(U1-5V-Pad14) -> 5V
Routing:
- net Net-(J1-VCC): track 106.2 -> 0.00 mm
- net 3V3: track 0.00 -> 87.9 mm
- net Net-(D1-A): track 0.00 -> 50.3 mm, vias 0 -> 1
- net GND: track 144.7 -> 190.1 mm
- net D0: track 41.9 -> 84.1 mm
- net 5V: track 0.00 -> 40.7 mm
- net D2: track 84.6 -> 50.2 mm
- net D3: track 55.4 -> 27.2 mm
- net D7: track 54.3 -> 72.6 mm
- net D1: track 73.7 -> 60.3 mm
- net Net-(J5-B-): track 44.2 -> 33.6 mm
- net Net-(J6-V0): track 37.9 -> 48.3 mm
- net B+: track 40.5 -> 48.1 mm
- net D10: track 68.8 -> 61.3 mm
- net D9: track 60.9 -> 68.2 mm
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
Commit message: edit pcb, update readme
Parts:
- moved J5 0.25 mm to (116.8, 31.0)
- turned J6 to 180 degrees
- turned U1 to 180 degrees
Routing:
- net GND: track 190.1 -> 130.7 mm, vias 0 -> 1
- net D0: track 84.1 -> 33.2 mm
- net D6: track 40.3 -> 68.4 mm
- net D8: track 60.3 -> 86.0 mm
- net 3V3: track 87.9 -> 62.5 mm
- net Net-(D1-A): track 50.3 -> 25.8 mm, vias 1 -> 0
- net 5V: track 40.7 -> 21.2 mm
- net D4: track 22.3 -> 38.9 mm
- net D5: track 27.1 -> 42.5 mm
- net D9: track 68.2 -> 54.8 mm
- net D10: track 61.3 -> 52.6 mm
- net D7: track 72.6 -> 63.9 mm
- net D2: track 50.2 -> 58.4 mm
- net B+: track 48.1 -> 42.0 mm, vias 0 -> 2
- net Net-(J6-V0): track 48.3 -> 43.9 mm
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